File: General Gantry/Gantry Hub V2/Gantry Hub V2 PCB/Gantry Hub V2 PCB.kicad_sch (KiCad schematic)
At the start: 0 parts

Commit message: Updates to gantry hub V2
Parts:
- added C1: 100uF, symbol Device:C_Polarized
- added C2: 330uF, symbol Device:C_Polarized
- added C5, C7: 10uF, symbol Device:C
- added C6, C8: 0.1uF, symbol Device:C
- added D1: 11DQ06, symbol Device:D_Schottky
- added J1: Conn_01x02_Socket, symbol Connector:Conn_01x02_Socket
- added J3: DIN-8, symbol Connector:DIN-8
- added J4, J5: DIN-4, symbol Connector:DIN-4
- added L1: 330uH, symbol Device:L
- added R2, R3: 10k, symbol Device:R
- added R4, R5: 14.3k, symbol Device:R
- added U2: SC0915, lib_footprints:CONN_4840-6004-CP_3MM, symbol 2026-07-30_18-39-20:SC0915
- added U3: LM2575-5.0BT, Package_TO_SOT_THT:TO-220-5_Vertical, symbol Regulator_Switching:LM2575-5.0BT
- added U5: LM358, symbol Amplifier_Operational:LM358
- added U6: MCP4802, symbol Analog_DAC:MCP4802
- added U7: SN74AHCT125N, Package_DIP:DIP-14_W7.62mm_Socket_LongPads, symbol Gantry Hub V2:SN74AHCT125N
Connections:
- new net: R3.1, R5.1, U5.6 (-)
- new net: U5.5 (+), U6.6 (VB)
- new net: U5.3 (+), U6.8 (VA)
- new net: R2.1, R4.1, U5.2 (-)
- new net: L1.1, U3.2 (OUT)
- new net +24V: C1.1, C7.2, C8.2, J1.1 (Pin_1), J4.1, J5.1, U3.1 (VIN), U5.8 (V+)
- new net +5V: C2.1, C5.1, C6.1, D1.1 (K), L1.2, U2.39 (VSYS), U3.4 (FB), U6.1 (Vdd), U7.14 (VCC)
- new net ANALOG_OUT_1: J4.2, R4.2, U5.1
- new net ANALOG_OUT_2: J5.2, R5.2, U5.7
- new net DAC_~{CS}: U6.2 (~{CS})
- new net DISPENSE_ENABLE: U7.2 (1A)
- new net DISPENSE_ENABLE_OUT: J3.1, U7.3 (1Y)
- new net GND: C1.2, C2.2, C5.2, C6.2, C7.1, C8.1, D1.2 (A), J1.2 (Pin_2), J3.2, J4.3, J5.3, R2.2, R3.2, U2.13 (GND), U2.18 (GND), U2.23 (GND), U2.28 (GND), U2.3 (GND), U2.38 (GND), U2.8 (GND), U3.3 (GND), U3.5 (~{ON}/OFF), U5.4 (V-), U6.5 (~{LDAC}), U6.7 (Vss), U7.1 (1~{OE}), U7.10 (3~{OE}), U7.13 (4~{OE}), U7.4 (2~{OE}), U7.7 (GND)
- new net SPI_SCK: U6.3 (SCK)
- new net SPI_SDI: U6.4 (SDI)
- no-connect marks 0 -> 24
Other:
- note added: "DAC Output range is 0V to 4.096V (in high-gain mode) Analog output range should be 0V to 10V Require op-amp gain of 10/4.096=2.44 Non-inverting topology gain is G= 1 + R_{F} / R_{g} Choose R_{F} = 14.3k , R_{g} = 10.0k"
- note added: "Dispenser Plug"
- note added: "Key Features: - Solenoid valve control for 4x 16-channel vacuum manifolds - Control of fluid dispenser - Source analog voltage to control gantry-camera light, extra ouput channels? - Sink analog voltages for vacuum pressure monitor. Anything else?"
- note added: "Level translator 3.3V->5V Tie unused inputs low."
- note added: "Microscope Light Plug & Spare"
- note removed: "https://www.digikey.com/en/products/detail/microchip-technology/MCP23017T-E-SO/964184 https://www.digikey.com/en/products/detail/panasonic-industry/AQY282EH/646349"

Commit message: Finish schematic & begin layout of Hub V2
Parts:
- C1: footprint (none) -> Capacitor_THT:CP_Radial_D8.0mm_P3.50mm; Digikey (none) -> 1189-2330-ND
- C2: footprint (none) -> Capacitor_THT:CP_Radial_D8.0mm_P3.50mm; Digikey (none) -> 1189-1251-ND
- C5, C6, C7, C8: footprint (none) -> Capacitor_SMD:C_1206_3216Metric_Pad1.33x1.80mm_HandSolder
- D1: footprint (none) -> Diode_THT:D_DO-41_SOD81_P7.62mm_Horizontal; Digikey (none) -> 1655-11DQ06CT-ND
- J1: footprint (none) -> lib_footprints:CONN_SDA_43255-00xx_02_MOL; Digikey (none) -> WM23264-ND
- J3: footprint (none) -> lib_footprints:CUI_SDF-80J; Digikey (none) -> CP-7080-ND
- J4, J5: footprint (none) -> lib_footprints:CUI_SDF-40J; Digikey (none) -> CP-7040-ND
- L1: footprint (none) -> lib_footprints:IND_PE-526xx_V_PUL; Digikey (none) -> 553-1558-5-ND
- R2, R3, R4, R5: footprint (none) -> Resistor_SMD:R_1206_3216Metric_Pad1.30x1.75mm_HandSolder
- U2: footprint lib_footprints:CONN_4840-6004-CP_3MM -> lib_footprints:SC0915
- U3: value LM2575-5.0BT -> LM2575-5.0WT; Digikey (none) -> 576-1516-5-ND
- U5: footprint (none) -> Package_DIP:DIP-8_W7.62mm_Socket_LongPads; Digikey (none) -> 296-1395-5-ND
- U6: footprint (none) -> Package_DIP:DIP-8_W7.62mm_Socket_LongPads; Digikey (none) -> MCP4802-E/P-ND
Connections:
- net GND: now also J3.S1, J3.S2, J4.S1, J4.S2, J5.S1, J5.S2
Other:
- note added: "DAC Output range is 0V to 4.096V (in high-gain mode) Analog output range should be 0V to 10V Require op-amp gain of 10/4.096=2.44 Non-inverting topology gain is G= 1 + R_{F} / R_{g} Choose R_{F} = 14.3k , R_{g} = 10.0k Socket in Digikey: 1175-1475-ND"
- note added: "Level translator 3.3V->5V Tie unused inputs low. Socket in Digikey: 1175-1476-ND"
- note added: "Socket in Digikey: 1175-1475-ND"
- note removed: "DAC Output range is 0V to 4.096V (in high-gain mode) Analog output range should be 0V to 10V Require op-amp gain of 10/4.096=2.44 Non-inverting topology gain is G= 1 + R_{F} / R_{g} Choose R_{F} = 14.3k , R_{g} = 10.0k"
- note removed: "Level translator 3.3V->5V Tie unused inputs low."

Commit message: Finalizes GH V2 part placement, about 60-75 percent done with routing
Parts:
- added J7, J8: Barrel_Jack, lib_footprints:CUI PJ-037A, symbol Connector:Barrel_Jack
Connections:
- net +24V: now also J7.1, J8.1
- net GND: now also J7.2, J8.2
Other:
- note added: "Mount to PCB w/ 2x 20-pin female headers, digikey 732-61302011821-ND 2x soldered 20-pin male headers, digikey SAM10260-ND"
- moved on the sheet: C1, C2, D1, J1, L1, U3

Commit message: Finishes V2.0 of gantry hub box
Parts:
- removed J4, J5: DIN-4, lib_footprints:CUI_SDF-40J, symbol Connector:DIN-4
- added D2: 11DQ06, Diode_THT:D_A-405_P7.62mm_Horizontal, symbol Device:D_Schottky
- added J4, J5: Mini-DIN-4, lib_footprints:CUI_MD-40SM, symbol Connector:Mini-DIN-4
- C5, C7: Digikey (none) -> 311-1959-1-ND
- C6, C8: Digikey (none) -> 311-1179-1-ND
- J7, J8: Digikey (none) -> CP-037A-ND
- R2, R3: Digikey (none) -> YAG3805CT-ND
- R4, R5: Digikey (none) -> 13-AC1206FR-0714K3LCT-ND
- U2: Digikey (none) -> 2648-SC0915CT-ND
- U7: Digikey (none) -> 296-4655-5-ND
Connections:
- net DISPENSE_ENABLE is gone; now on net D0: U7.2 (1A)
- net SPI_SCK is gone; now on net DAC_{SCK}: U6.3 (SCK)
- net SPI_SDI is gone; now on net DAC_{SDI}: U6.4 (SDI)
- net +24V: now also J4.1, J5.1
- net +5V: now also D2.2 (A); no longer U2.39 (VSYS)
- net ANALOG_OUT_1: now also J5.2
- net ANALOG_OUT_2: now also J4.2
- net DAC_~{CS}: now also U2.12 (UART1_RX/I2C0_SCL/SPI1_CSn/GP9)
- net GND: now also J4.3, J4.SHIELD, J5.3, J5.SHIELD
- net D3: now reaches U7.12 (4A)
- net D3: now also U2.9 (I2C1_SDA/SPI0_SCK/GP6)
- net D1: now reaches U7.5 (2A)
- net D1: now also U2.11 (UART1_TX/I2C0_SDA/SPI1_RX/GP8)
- net D2: now reaches U7.9 (3A)
- net D2: now also U2.10 (I2C1_SCL/SPI0_TX/GP7)
- net MNFLD-~{SRCLR}: now reaches U2.1 (UART0_TX/I2C0_SDA/SPI0_RX/GP0)
- net DAC_{SCK}: now reaches U2.14 (I2C1_SDA/SPI1_SCK/GP10)
- net DAC_{SDI}: now reaches U2.15 (I2C1_SCL/SPI1_TX/GP11)
- net MNFLD-DISABLE: now reaches U2.2 (UART0_RX/I2C0_SCL/GPI0_CSn/GP1)
- net MNFLD-S_{CK}: now reaches U2.4 (I2C1_SDA/SPI0_SCK/GP2)
- net MNFLD-S_{IN}: now reaches U2.5 (I2C1_SCL/SPI0_TX/GP3)
- net MNFLD-R_{CK}: now reaches U2.6 (UART1_TX/I2C0_SDA/SPI0_RX/GP4)
- net D0: now reaches U2.7 (UART1_RX/I2C0_SCL/SPI0_CSn/GP5)
- new net: D2.1 (K), U2.39 (VSYS)
Other:
- note added: "Digikey parts list: https://www.digikey.com/en/mylists/list/8ZQ23FV3C8"
- note added: "Mount to PCB w/ 2x 20-pin female headers, digikey 732-61302011821-ND 2x soldered 20-pin male headers, digikey 612-TS-120-T-A-ND"
- note added: "Schottky diode to avoid USB back-feeding power to system"
- note removed: "Mount to PCB w/ 2x 20-pin female headers, digikey 732-61302011821-ND 2x soldered 20-pin male headers, digikey SAM10260-ND"
- title: (none) -> Gantry Hub PCB
